File: Hardware_Board/RASPBERRY PI.kicad_sch (KiCad schematic)
At the start: 2 parts, among them U2 RASPBERRY_PI_4B_4GB

Commit message: esc board updated
Parts:
- added D28: LED, symbol Device:LED
- added J10, J11, J12, J9: Conn_01x03, symbol Connector_Generic:Conn_01x03
- added R28: 1K, symbol Device:R
Connections:
- net +5V: now also J10.2 (Pin_2), J11.2 (Pin_2), J12.2 (Pin_2), J9.2 (Pin_2)
- net GND: now also D28.1 (K), J10.1 (Pin_1), J11.1 (Pin_1), J12.1 (Pin_1), J9.1 (Pin_1)
- net LED0: now also R28.1
- net SERVO0: now also J9.3 (Pin_3)
- net SERVO1: now also J10.3 (Pin_3)
- net SERVO2: now also J11.3 (Pin_3)
- net SERVO3: now also J12.3 (Pin_3)
- net SWCLK1: no longer U2.37 (GPIO26)
- net SWD1: no longer U2.40 (GPIO21)
- new net: D28.2 (A), R28.2
- new net SWCLK2: U2.37 (GPIO26)
- new net SWD2: U2.40 (GPIO21)
Other:
- note added: "Servo Connectors"
- note added: "Status LEDs"
