File: Hardware_Board/Switching.kicad_sch (KiCad schematic)
At the start: 50 parts, among them J1 Conn_01x02, J2 Conn_01x02, J3 Conn_01x02, J4 Conn_01x02, J7 Conn_01x02, Q1 ZXMN3A14F, Q2 ZXMN3A14F, Q3 ZXMN3A14F, Q4 ZXMN3A14F, Q7 ZXMN3A14F

Commit message: esc board updated
Parts:
- added C5, C6, C8: 2.2uF+/35V+, Capacitor_SMD:C_0805_2012Metric, symbol Adafruit MOSFET Driver STEMMA Breakout-eagle-import:CAP_CERAMIC0805-NOOUTLINE
- added D15, D18, D24: LED_Red, LED_SMD:LED_0603_1608Metric, symbol Device:LED
- added D16, D22, D25: LED_Green, LED_SMD:LED_0603_1608Metric, symbol Device:LED
- added D17, D23, D26: SM4002, Diode_SMD:D_SOD-123F, symbol Diode:SM4002
- added F1, F7, F9: Fuse, Fuse:Fuse_0805_2012Metric, symbol Device:Fuse
- added J5, J6, J8: Conn_01x02, Rpi_Pico_header:Molex_Micro-Latch_53253-0270_1x02_P2.00mm_Vertical_3D_model, symbol Connector_Generic:Conn_01x02
- added Q5, Q6, Q8: ZXMN3A14F, Package_TO_SOT_SMD:SOT-23, symbol Transistor_FET:ZXMN3A14F
- added R15, R16, R17, R18, R22, R23, R24, R25, R26: 10k, Resistor_SMD:R_0805_2012Metric, symbol Adafruit MOSFET Driver STEMMA Breakout-eagle-import:RESISTOR_0603_NOOUT
Connections:
- net +5V: now also F1.2, F7.2, F9.2
- net GND: now also C5.2, C6.2, C8.2, D15.1 (K), D16.1 (K), D18.1 (K), D22.1 (K), D24.1 (K), D25.1 (K), Q5.2 (S), Q6.2 (S), Q8.2 (S), R17.1, R23.1, R26.1
- removed net GPIO (): Q1.1 (G), Q2.1 (G), Q3.1 (G), Q4.1 (G), Q7.1 (G), R1.2, R10.2, R12.2, R19.2, R21.2, R3.2, R4.2, R6.2, R7.2, R9.2
- new net: C5.1, D17.1 (K), F1.1, J5.1 (Pin_1), R16.2
- new net: D15.2 (A), R15.1
- new net: D25.2 (A), R25.1
- new net: C6.1, D23.1 (K), F7.1, J6.1 (Pin_1), R22.2
- new net: D16.2 (A), R16.1
- new net: D22.2 (A), R22.1
- new net: D26.2 (A), J8.2 (Pin_2), Q8.3 (D)
- new net: D17.2 (A), J5.2 (Pin_2), Q5.3 (D)
- new net: D24.2 (A), R24.1
- new net: C8.1, D26.1 (K), F9.1, J8.1 (Pin_1), R25.2
- new net: D23.2 (A), J6.2 (Pin_2), Q6.3 (D)
- new net: D18.2 (A), R18.1
- new net SW0: Q1.1 (G), R1.2, R3.2
- new net SW1: Q2.1 (G), R4.2, R6.2
- new net SW2: Q3.1 (G), R7.2, R9.2
- new net SW3: Q7.1 (G), R19.2, R21.2
- new net SW4: Q4.1 (G), R10.2, R12.2
- new net SW5: Q5.1 (G), R15.2, R17.2
- new net SW6: Q6.1 (G), R18.2, R23.2
- new net SW7: Q8.1 (G), R24.2, R26.2
Other:
- moved on the sheet: C4, D10, D11, D12, F5, J4, Q4, R10, R11, R12
