File: Backplane_Board/Voltage Level ADC.kicad_sch (KiCad schematic)
At the start: 11 parts, among them U6 ADS1115IDGS

Commit message: add rerevised esc board and rough backplane schmatic
Other:
- company: (none) -> Cabrillo Robtics
- title: (none) -> Backplane_Board
Changed lines of the file:
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@@
 	(generator_version "8.0")
 	(paper "A4")
+	(title_block
+		(title "Backplane_Board")
+		(date "2024-09-30")
+		(rev "1")
+		(company "Cabrillo Robtics")
+		(comment 1 "LaserShark Backplane PCB")
+	)
 	(junction
 		(at 63.5 67.31)
