File: Backplane_Board/Backplane_Board.kicad_sch (KiCad schematic)
At the start: 15 parts, among them J1 XT60, J2 XT60, J3 Conn_01x02_Pin, Q1 FDMS86163P, Q2 FDMS86163P, U1 ZXTR2005ZQ-13

Commit message: added gerber
Parts:
- R2: value 620 -> 1k
- U1: footprint ZXTR2005ZQ-13:SOT-89_4P5X2P45_DIO-M -> Package_TO_SOT_SMD:SOT-89-3_Handsoldering
Changed lines of the file:
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@@
 			)
 		)
-		(property "Footprint" "ZXTR2005ZQ-13:SOT-89_4P5X2P45_DIO-M"
+		(property "Footprint" "Package_TO_SOT_SMD:SOT-89-3_Handsoldering"
 			(at 82.042 128.143 0)
 			(effects
@@
 			)
 		)
-		(property "Value" "620"
+		(property "Value" "1k"
 			(at 149.86 158.7499 0)
 			(effects
