File: Backplane_Board/Power_Connectors.kicad_sch (KiCad schematic)
At the start: 27 parts, among them J10 Conn_01x02_Pin, J11 Conn_01x02_Pin, J12 Conn_01x02_Pin, J13 Conn_01x02_Pin, J14 Conn_01x02_Pin, J15 Conn_01x02_Pin, J16 Conn_01x02_Pin, J17 Conn_01x02_Pin, J18 Conn_01x02_Pin, J19 Conn_01x02_Pin, J20 Conn_01x02_Pin, J21 Conn_01x02_Pin, J22 Conn_01x02_Pin, J23 Conn_01x02_Pin, J24 Conn_01x02_Pin, J6 Conn_01x02_Pin, J7 Conn_01x02_Pin, J8 Conn_01x02_Pin, J9 Conn_01x02_Pin, U5 PKU3511SPI

Commit message: derat nest ifcation
Parts:
- removed C22: 330 uF, 220UF CAP:CAP_16SVPG330MX, symbol Device:C_Polarized_Small_US
- removed J19, J6, J8, J9: Conn_01x02_Pin, Connector_AMASS:AMASS_XT30U-M_1x02_P5.0mm_Vertical, symbol Connector:Conn_01x02_Pin
- added J11, J12, J13, J14, J15, J16: Conn_01x02_Pin, Connector_AMASS:AMASS_XT30U-M_1x02_P5.0mm_Vertical, symbol Connector:Conn_01x02_Pin
- C19: renamed from C20; footprint 220UF CAP:CAP_16SVPG330MX -> Capacitor_SMD:CP_Elec_6.3x7.7
- C20: renamed from C21; footprint 220UF CAP:CAP_16SVPG330MX -> Capacitor_SMD:CP_Elec_6.3x7.7
- J19: renamed from J14; footprint TerminalBlock:TerminalBlock_Xinya_XY308-2.54-2P_1x02_P2.54mm_Horizontal -> TerminalBlock_4Ucon:TerminalBlock_4Ucon_1x02_P3.50mm_Horizontal
- J20: renamed from J15; footprint TerminalBlock:TerminalBlock_Xinya_XY308-2.54-2P_1x02_P2.54mm_Horizontal -> TerminalBlock_4Ucon:TerminalBlock_4Ucon_1x02_P3.50mm_Horizontal
- J21: renamed from J16; footprint TerminalBlock:TerminalBlock_Xinya_XY308-2.54-2P_1x02_P2.54mm_Horizontal -> TerminalBlock_4Ucon:TerminalBlock_4Ucon_1x02_P3.50mm_Horizontal
- J22: renamed from J20; footprint TerminalBlock_4Ucon:TerminalBlock_4Ucon_1x02_P3.50mm_Horizontal -> Connector_AMASS:AMASS_XT30U-M_1x02_P5.0mm_Vertical
- J23: renamed from J21; footprint TerminalBlock_4Ucon:TerminalBlock_4Ucon_1x02_P3.50mm_Horizontal -> Connector_AMASS:AMASS_XT30U-M_1x02_P5.0mm_Vertical
- J24: renamed from J22; footprint TerminalBlock_4Ucon:TerminalBlock_4Ucon_1x02_P3.50mm_Horizontal -> Connector_AMASS:AMASS_XT30U-M_1x02_P5.0mm_Vertical
- J25: renamed from J23; footprint TerminalBlock_4Ucon:TerminalBlock_4Ucon_1x02_P3.50mm_Horizontal -> Connector_AMASS:AMASS_XT30U-M_1x02_P5.0mm_Vertical
- J6: renamed from J11; footprint TerminalBlock:TerminalBlock_Xinya_XY308-2.54-2P_1x02_P2.54mm_Horizontal -> TerminalBlock_4Ucon:TerminalBlock_4Ucon_1x02_P3.50mm_Horizontal
- J7: renamed from J12; footprint TerminalBlock:TerminalBlock_Xinya_XY308-2.54-2P_1x02_P2.54mm_Horizontal -> TerminalBlock_4Ucon:TerminalBlock_4Ucon_1x02_P3.50mm_Horizontal
- J8: renamed from J13; footprint TerminalBlock:TerminalBlock_Xinya_XY308-2.54-2P_1x02_P2.54mm_Horizontal -> TerminalBlock_4Ucon:TerminalBlock_4Ucon_1x02_P3.50mm_Horizontal
- R20: footprint Resistor_SMD:R_1206_3216Metric_Pad1.30x1.75mm_HandSolder -> Resistor_SMD:R_0805_2012Metric_Pad1.20x1.40mm_HandSolder
- renumbered J24 to J26, J7 to J9
Connections:
- net 12V_ESC: now also J11.2 (Pin_2), J12.2 (Pin_2), J13.2 (Pin_2), J14.2 (Pin_2), J15.2 (Pin_2), J16.2 (Pin_2)
- net GND: now also J11.1 (Pin_1), J12.1 (Pin_1), J13.1 (Pin_1), J14.1 (Pin_1), J15.1 (Pin_1), J16.1 (Pin_1)
Other:
- moved on the sheet: J19, J20, J21, J22, J23, J24, J25, J6, J7, J8, J9

Commit message: add 3d modules and clean up footprints
Parts:
- J10, J11, J12, J13, J14, J15, J16, J17, J18, J22, J23, J24, J25, J9: footprint Connector_AMASS:AMASS_XT30U-M_1x02_P5.0mm_Vertical -> XT30U-F_IW:AMASS_XT30U-M_1x02_P5.0mm_Vertical_IW_3d
- J19, J20, J21, J6, J7, J8: footprint TerminalBlock_4Ucon:TerminalBlock_4Ucon_1x02_P3.50mm_Horizontal -> 3.5_pitch_2x2_block:TerminalBlock_4Ucon_1x02_P3.50mm_Horizontal_updated
Changed lines of the file:
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@@
 			)
 		)
-		(property "Footprint" "TerminalBlock_4Ucon:TerminalBlock_4Ucon_1x02_P3.50mm_Horizontal"
+		(property "Footprint" "3.5_pitch_2x2_block:TerminalBlock_4Ucon_1x02_P3.50mm_Horizontal_updated"
 			(at 95.25 133.35 0)
 			(effects
@@
 			)
 		)
-		(property "Footprint" "Connector_AMASS:AMASS_XT30U-M_1x02_P5.0mm_Vertical"
+		(property "Footprint" "XT30U-F_IW:AMASS_XT30U-M_1x02_P5.0mm_Vertical_IW_3d"
 			(at 196.85 125.73 0)
 			(effects
@@
 			)
 		)
-		(property "Footprint" "Connector_AMASS:AMASS_XT30U-M_1x02_P5.0mm_Vertical"
+		(property "Footprint" "XT30U-F_IW:AMASS_XT30U-M_1x02_P5.0mm_Vertical_IW_3d"
 			(at 260.35 125.73 0)
 			(effects
@@
 			)
 		)
-		(property "Footprint" "Connector_AMASS:AMASS_XT30U-M_1x02_P5.0mm_Vertical"
+		(property "Footprint" "XT30U-F_IW:AMASS_XT30U-M_1x02_P5.0mm_Vertical_IW_3d"
 			(at 273.05 125.73 0)
 			(effects
@@
 			)
 		)
-		(property "Footprint" "TerminalBlock_4Ucon:TerminalBlock_4Ucon_1x02_P3.50mm_Horizontal"
+		(property "Footprint" "3.5_pitch_2x2_block:TerminalBlock_4Ucon_1x02_P3.50mm_Horizontal_updated"
 			(at 81.28 118.11 0)
 			(effects
@@
 			)
 		)
-		(property "Footprint" "Connector_AMASS:AMASS_XT30U-M_1x02_P5.0mm_Vertical"
+		(property "Footprint" "XT30U-F_IW:AMASS_XT30U-M_1x02_P5.0mm_Vertical_IW_3d"
 			(at 158.75 125.73 0)
 			(effects
@@
 			)
 		)
-		(property "Footprint" "Connector_AMASS:AMASS_XT30U-M_1x02_P5.0mm_Vertical"
+		(property "Footprint" "XT30U-F_IW:AMASS_XT30U-M_1x02_P5.0mm_Vertical_IW_3d"
 			(at 99.06 167.64 0)
 			(effects
@@
 			)
 		)
-		(property "Footprint" "TerminalBlock_4Ucon:TerminalBlock_4Ucon_1x02_P3.50mm_Horizontal"
+		(property "Footprint" "3.5_pitch_2x2_block:TerminalBlock_4Ucon_1x02_P3.50mm_Horizontal_updated"
 			(at 100.33 118.11 0)
 			(effects
@@
 			)
 		)
-		(property "Footprint" "Connector_AMASS:AMASS_XT30U-M_1x02_P5.0mm_Vertical"
+		(property "Footprint" "XT30U-F_IW:AMASS_XT30U-M_1x02_P5.0mm_Vertical_IW_3d"
 			(at 234.95 125.73 0)
 			(effects
@@
 			)
 		)
-		(property "Footprint" "Connector_AMASS:AMASS_XT30U-M_1x02_P5.0mm_Vertical"
+		(property "Footprint" "XT30U-F_IW:AMASS_XT30U-M_1x02_P5.0mm_Vertical_IW_3d"
 			(at 59.69 167.64 0)
 			(effects
@@
 			)
 		)
-		(property "Footprint" "Connector_AMASS:AMASS_XT30U-M_1x02_P5.0mm_Vertical"
+		(property "Footprint" "XT30U-F_IW:AMASS_XT30U-M_1x02_P5.0mm_Vertical_IW_3d"
 			(at 184.15 125.73 0)
 			(effects
@@
 			)
 		)
-		(property "Footprint" "Connector_AMASS:AMASS_XT30U-M_1x02_P5.0mm_Vertical"
+		(property "Footprint" "XT30U-F_IW:AMASS_XT30U-M_1x02_P5.0mm_Vertical_IW_3d"
 			(at 80.01 167.64 0)
 			(effects
@@
 			)
 		)
-		(property "Footprint" "Connector_AMASS:AMASS_XT30U-M_1x02_P5.0mm_Vertical"
+		(property "Footprint" "XT30U-F_IW:AMASS_XT30U-M_1x02_P5.0mm_Vertical_IW_3d"
 			(at 116.84 167.64 0)
 			(effects
@@
 			)
 		)
-		(property "Footprint" "Connector_AMASS:AMASS_XT30U-M_1x02_P5.0mm_Vertical"
+		(property "Footprint" "XT30U-F_IW:AMASS_XT30U-M_1x02_P5.0mm_Vertical_IW_3d"
 			(at 247.65 125.73 0)
 			(effects
@@
 			)
 		)
-		(property "Footprint" "Connector_AMASS:AMASS_XT30U-M_1x02_P5.0mm_Vertical"
+		(property "Footprint" "XT30U-F_IW:AMASS_XT30U-M_1x02_P5.0mm_Vertical_IW_3d"
 			(at 209.55 125.73 0)
 			(effects
@@
 			)
 		)
-		(property "Footprint" "Connector_AMASS:AMASS_XT30U-M_1x02_P5.0mm_Vertical"
+		(property "Footprint" "XT30U-F_IW:AMASS_XT30U-M_1x02_P5.0mm_Vertical_IW_3d"
 			(at 222.25 125.73 0)
 			(effects
@@
 			)
 		)
-		(property "Footprint" "Connector_AMASS:AMASS_XT30U-M_1x02_P5.0mm_Vertical"
+		(property "Footprint" "XT30U-F_IW:AMASS_XT30U-M_1x02_P5.0mm_Vertical_IW_3d"
 			(at 171.45 125.73 0)
 			(effects
@@
 			)
 		)
-		(property "Footprint" "TerminalBlock_4Ucon:TerminalBlock_4Ucon_1x02_P3.50mm_Horizontal"
+		(property "Footprint" "3.5_pitch_2x2_block:TerminalBlock_4Ucon_1x02_P3.50mm_Horizontal_updated"
 			(at 76.2 133.35 0)
 			(effects
@@
 			)
 		)
-		(property "Footprint" "TerminalBlock_4Ucon:TerminalBlock_4Ucon_1x02_P3.50mm_Horizontal"
+		(property "Footprint" "3.5_pitch_2x2_block:TerminalBlock_4Ucon_1x02_P3.50mm_Horizontal_updated"
 			(at 114.3 133.35 0)
 			(effects
@@
 			)
 		)
-		(property "Footprint" "TerminalBlock_4Ucon:TerminalBlock_4Ucon_1x02_P3.50mm_Horizontal"
+		(property "Footprint" "3.5_pitch_2x2_block:TerminalBlock_4Ucon_1x02_P3.50mm_Horizontal_updated"
 			(at 119.38 118.11 0)
 			(effects

Commit message: added gerber
Parts:
- R20: value 620 -> 1k
Changed lines of the file:
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@@
 			)
 		)
-		(property "Value" "620"
+		(property "Value" "1k"
 			(at 271.78 50.7999 0)
 			(effects
